Commit message: changes for new moveit config

File: icl_ur5_setup_description/robots/ur5_robotiq_140_joint_limited_linear.xacro (robot description, xacro)
@@ -3,13 +3,15 @@
   <!-- include macros for UR5 and the Robotiq eef model -->
   <xacro:include filename="$(find ur_description)/urdf/common.gazebo.xacro" />
-  <xacro:include filename="$(find ur_description)/urdf/ur5.urdf.xacro" />
-  <xacro:include filename="$(find icl_ur5_setup_description)/urdf/robotiq_arg2f_140_model_macro.xacro" />
-  <xacro:include filename="$(find icl_ur5_setup_description)/urdf/robotiq_fts300.urdf.xacro" />
-  <xacro:include filename="$(find cougarbot)/urdf/cougarbot_short.urdf.xacro" />
-  <xacro:include filename="$(find ypc_simulation)/dwq_model/urdf/oven.xacro"/>
-  <xacro:include filename="$(find ypc_simulation)/dwq_model/urdf/ypc_slide_vertical.xacro"/>
+  <xacro:include filename="$(find ypc_simulation)/urdf/ur5_with_slide_base.xacro" />
+  <!-- <xacro:include filename="$(find ur_description)/urdf/ur5.urdf.xacro" /> -->
+  <!-- <xacro:include filename="$(find icl_ur5_setup_description)/urdf/robotiq_arg2f_140_model_macro.xacro" />
+  <xacro:include filename="$(find icl_ur5_setup_description)/urdf/robotiq_fts300.urdf.xacro" /> -->
+  <!-- <xacro:include filename="$(find cougarbot)/urdf/cougarbot_short.urdf.xacro" /> -->
+  <xacro:include filename="$(find ypc_simulation)/urdf/oven.xacro"/>
+  <xacro:include filename="$(find ypc_simulation)/urdf/ypc_slide_vertical.xacro"/>
+  <xacro:include filename="$(find ypc_simulation)/urdf/liquid_robot.xacro"/>
   <xacro:macro name="ur5_with_gripper_joint_limited" params="prefix">
     <!-- arm -->
-    <xacro:ur5_robot prefix="${prefix}" joint_limited="true"
+    <!-- <xacro:ur5_robot prefix="${prefix}" joint_limited="true"
       shoulder_pan_lower_limit="${-3*pi/4}" shoulder_pan_upper_limit="${pi/2}"
       shoulder_lift_lower_limit="${-pi*7/8}" shoulder_lift_upper_limit="${-pi/8}"
@@ -18,5 +20,5 @@
       wrist_2_lower_limit="${-pi}" wrist_2_upper_limit="${pi}"
       wrist_3_lower_limit="${-pi}" wrist_3_upper_limit="${pi}"
-    />
+    /> -->
 <!-- the white base  -->
     <link name="world" />
@@ -24,20 +26,24 @@
       <parent link= "world" />
       <child link = "linear_base_link" />
-      <origin xyz="0.0 0.0 1.5" rpy="0.0 ${pi} 0.0" />
+      <origin xyz="0.0 0.0 2.5" rpy="0.0 ${pi} 0.0" />
     </joint>
 <!-- only arm  -->
-    <joint name="fixed_link_robot_base" type="fixed">
+    <!-- <joint name="fixed_link_robot_base" type="fixed">
       <parent link= "slide_plate" />
       <child link = "${prefix}base_link" />
       <origin xyz="0.0 0.0 0.02" rpy="0.0 0.0 0.0" />
-    </joint>
+    </joint> -->
     <!-- ypc oven -->
     <xacro:ypc_oven parent="world"/>
+    <!-- ypc slide vertical -->
     <xacro:ypc_cupboard_dwq parent="world"/>
-    <!--force torque sensor-->
-    <xacro:robotiq_fts150 prefix="" parent="ee_link" >
+    <!-- ypc liquid robot -->
+    <xacro:ypc_liquid_robot parent="world"/>
+    <!-- force torque sensor -->
+    <!-- <xacro:robotiq_fts150 prefix="" parent="ee_link" >
       <origin xyz="0.009 0 0 " rpy="-${pi/2} 0 -${pi/2}"/>
-    </xacro:robotiq_fts150>
+    </xacro:robotiq_fts150> -->
    <!-- gripper -->
+<!--
     <xacro:robotiq_arg2f_140 prefix="${prefix}" />
     <joint name="ur5_ee_link_gripper_base" type="fixed">
@@ -51,5 +57,5 @@
       <child link = "${prefix}tool" />
       <origin xyz=" 0.00 0.0 0.2" rpy="0.0 0.0 0.0" />
-    </joint>
+    </joint> -->
   </xacro:macro>
   <xacro:ur5_with_gripper_joint_limited prefix=""/>
